Commit message: joint state publisher working with rviz on drivebase

File: ante_description/robots/ante.urdf.xacro (robot description, xacro)
@@ -7,5 +7,5 @@
     <!-- create drivebase using macro -->
     <xacro:drivebase parent="base_link">
-        <origin xyz="0 0 0" rpy="0 0 0"/>
+        <origin xyz="0 0 1" rpy="0 0 0"/>
     </xacro:drivebase>
 </robot>

File: ante_description/urdf/drivebase.xacro (robot description, xacro)
@@ -6,5 +6,5 @@
     <parent link="${parent}"/>
     <child link="chassis_link"/>
-    <xacro:insert_block name="origin" />
+    <!-- <xacro:insert_block name="origin" /> -->
   </joint>
   <!-- wheel joints -->

Commit message: added ducket and solenoids to urdf

File: ante_description/robots/ante.urdf.xacro (robot description, xacro)
@@ -3,9 +3,18 @@
     <!-- include Files -->
     <xacro:include filename="$(find ante_description)/urdf/drivebase.xacro" />
+    <xacro:include filename="$(find ante_description)/urdf/ducket.xacro" />
+    <xacro:include filename="$(find ante_description)/urdf/solenoids.xacro" />
     <!-- create base_link -->
     <link name="base_link" />
     <!-- create drivebase using macro -->
     <xacro:drivebase parent="base_link">
-        <origin xyz="0 0 1" rpy="0 0 0"/>
+        <origin xyz="0 0 0" rpy="0 0 0"/>
     </xacro:drivebase>
+    <!-- create ducket and fasten to defined point -->
+    <xacro:ducket parent="base_link">
+        <origin xyz="0 -0.03 0.01" rpy="0 0 0"/>
+    </xacro:ducket>
+    <xacro:solenoids parent="base_link">
+        <origin xyz="-0.029 0.172 0.026" rpy="0 0 0"/>
+    </xacro:solenoids>
 </robot>

Commit message: started implementing mecanum controller

File: ante_description/robots/ante.urdf.xacro (robot description, xacro)
@@ -5,4 +5,5 @@
     <xacro:include filename="$(find ante_description)/urdf/ducket.xacro" />
     <xacro:include filename="$(find ante_description)/urdf/solenoids.xacro" />
+    <!-- <xacro:include filename="$(find ante_description)/urdf/ros2_control.xacro" /> -->
     <!-- create base_link -->
     <link name="base_link" />

File: ante_description/urdf/drivebase.xacro (robot description, xacro)
@@ -6,5 +6,5 @@
     <parent link="${parent}"/>
     <child link="chassis_link"/>
-    <!-- <xacro:insert_block name="origin" /> -->
+    <xacro:insert_block name="origin" />
   </joint>
   <!-- wheel joints -->
@@ -35,5 +35,5 @@
   <link name="chassis_link">
     <visual>
-      <origin xyz="0. 0. 0." rpy="0. 0. 0."/>
+      <origin xyz="0. 0. 5" rpy="0. 0. 0."/>
       <geometry>
         <mesh filename="package://ante_description/meshes/decimated_drivebase.obj" scale="1. 1. 1."/>

Commit message: added simple wheels and reader arm

File: ante_description/robots/ante.urdf.xacro (robot description, xacro)
@@ -1,21 +1,56 @@
 <?xml version="1.0" ?>
 <robot name="ante" xmlns:xacro="http://www.ros.org/wiki/xacro">
-    <!-- include Files -->
-    <xacro:include filename="$(find ante_description)/urdf/drivebase.xacro" />
-    <xacro:include filename="$(find ante_description)/urdf/ducket.xacro" />
-    <xacro:include filename="$(find ante_description)/urdf/solenoids.xacro" />
+    <!-- Include Files -->
+    <xacro:include filename="$(find ante_description)/parts/drivebase.xacro" />
+    <xacro:include filename="$(find ante_description)/parts/ducket.xacro" />
+    <xacro:include filename="$(find ante_description)/parts/solenoids.xacro" />
+    <xacro:include filename="$(find ante_description)/parts/simple_wheel.xacro" />
+    <xacro:include filename="$(find ante_description)/parts/reader_arm.xacro" />
     <!-- <xacro:include filename="$(find ante_description)/urdf/ros2_control.xacro" /> -->
     <!-- create base_link -->
     <link name="base_link" />
-    <!-- create drivebase using macro -->
     <xacro:drivebase parent="base_link">
         <origin xyz="0 0 0" rpy="0 0 0"/>
     </xacro:drivebase>
-    <!-- create ducket and fasten to defined point -->
-    <xacro:ducket parent="base_link">
-        <origin xyz="0 -0.03 0.01" rpy="0 0 0"/>
+    <xacro:simple_wheel
+        name="front_left"
+        parent="chassis_link"
+        flip="0"
+        pos_x="0.051"
+        pos_y="-0.070"
+        pos_z="0.0375"
+    />
+    <xacro:simple_wheel
+        name="front_right"
+        parent="chassis_link"
+        flip="1"
+        pos_x="-0.051"
+        pos_y="-0.070"
+        pos_z="0.0375"
+    />
+    <xacro:simple_wheel
+        name="rear_left"
+        parent="chassis_link"
+        flip="0"
+        pos_x="0.051"
+        pos_y="0.070"
+        pos_z="0.0375"
+    />
+    <xacro:simple_wheel
+        name="rear_right"
+        parent="chassis_link"
+        flip="1"
+        pos_x="-0.051"
+        pos_y="0.070"
+        pos_z="0.0375"
+    />
+    <xacro:ducket parent="chassis_link">
+        <origin xyz="0 -0.12025 0.041445" rpy="0 0 0"/>
     </xacro:ducket>
-    <xacro:solenoids parent="base_link">
-        <origin xyz="-0.029 0.172 0.026" rpy="0 0 0"/>
+    <xacro:solenoids parent="chassis_link">
+        <origin xyz="-0.029 0.052 0.0675" rpy="0 0 0"/>
     </xacro:solenoids>
+    <xacro:reader_arm parent="chassis_link">
+        <origin xyz="0 0 0.2" rpy="0 0 0" />
+    </xacro:reader_arm>
 </robot>
