Commit message: added knob wheel

File: ante_description/parts/drivebase.xacro (robot description, xacro)
@@ -14,87 +14,7 @@
         <mesh filename="package://ante_description/meshes/drivebase_frame_decimated.stl" scale="1. 1. 1."/>
       </geometry>
+      <material name="silver" />
     </visual>
   </link>
-  <!-- wheel joints -->
-  <!-- <joint name="front_left_axle" type="continuous">
-    <origin xyz="-0.051 0.103055 -0.055208" rpy="-1.5707964 0. 1.5707964"/>
-    <parent link="${parent}"/>
-    <child link="front_left_wheel"/>
-    <axis xyz="0. 0. 1."/>
-  </joint>
-  <joint name="front_right_axle" type="continuous">
-    <origin xyz="-0.111 0.042 -0.012" rpy="-1.5707964 0. -1.5707964"/>
-    <parent link="chassis_link"/>
-    <child link="front_right_wheel"/>
-    <axis xyz="0. 0. 1."/>
-  </joint>
-  <joint name="rear_left_axle" type="continuous">
-    <origin xyz="0.111 0.182 -0.012" rpy="-1.5707964 0. 1.5707964"/>
-    <parent link="chassis_link"/>
-    <child link="rear_left_wheel"/>
-    <axis xyz="0. 0. 1."/>
-  </joint>
-  <joint name="rear_right_axle" type="continuous">
-    <origin xyz="-0.111 0.182 -0.012" rpy="-1.5707964 0. -1.5707964"/>
-    <parent link="chassis_link"/>
-    <child link="rear_right_wheel"/>
-    <axis xyz="0. 0. 1."/>
-  </joint>
-  <link name="front_left_wheel">
-    <visual>
-      <origin xyz="0 0 0" rpy="1.5707964 1.5707964 0. "/>
-      <geometry>
-        <mesh filename="package://ante_description/meshes/simple_wheel.stl" scale="1. 1. 1."/>
-      </geometry>
-    </visual>
-    <collision>
-      <origin xyz="0. -0. 0.06" rpy="1.5707964 1.5707964 0. "/>
-      <geometry>
-        <mesh filename="package://ante_description/meshes/wheel.obj" scale="1. 1. 1."/>
-      </geometry>
-    </collision>
-  </link>
-  <link name="front_right_wheel">
-    <visual>
-      <origin xyz="-0. -0. 0.06" rpy="-0.3917964 1.5707964 0. "/>
-      <geometry>
-        <mesh filename="package://ante_description/meshes/wheel.obj" scale="1. 1. 1."/>
-      </geometry>
-    </visual>
-    <collision>
-      <origin xyz="-0. -0. 0.06" rpy="-0.3917964 1.5707964 0. "/>
-      <geometry>
-        <mesh filename="package://ante_description/meshes/wheel.obj" scale="1. 1. 1."/>
-      </geometry>
-    </collision>
-  </link>
-  <link name="rear_left_wheel">
-    <visual>
-      <origin xyz="0. -0. 0.02" rpy="-0.3917964 -1.5707964 0. "/>
-      <geometry>
-        <mesh filename="package://ante_description/meshes/wheel.obj" scale="1. 1. 1."/>
-      </geometry>
-    </visual>
-    <collision>
-      <origin xyz="0. -0. 0.02" rpy="-0.3917964 -1.5707964 0. "/>
-      <geometry>
-        <mesh filename="package://ante_description/meshes/wheel.obj" scale="1. 1. 1."/>
-      </geometry>
-    </collision>
-  </link>
-  <link name="rear_right_wheel">
-    <visual>
-      <origin xyz="-0. -0. 0.06" rpy="-0.3917964 1.5707964 0. "/>
-      <geometry>
-        <mesh filename="package://ante_description/meshes/wheel.obj" scale="1. 1. 1."/>
-      </geometry>
-    </visual>
-    <collision>
-      <origin xyz="-0. -0. 0.06" rpy="-0.3917964 1.5707964 0. "/>
-      <geometry>
-        <mesh filename="package://ante_description/meshes/wheel.obj" scale="1. 1. 1."/>
-      </geometry>
-    </collision>
-  </link> -->
 </xacro:macro>
 </robot>

File: ante_description/parts/reader_arm.xacro (robot description, xacro)
@@ -8,4 +8,5 @@
         <mesh filename="package://ante_description/meshes/reader_base.stl" scale="1. 1. 1."/>
       </geometry>
+      <material name="green" />
     </visual>
   </link>
@@ -25,4 +26,5 @@
         <mesh filename="package://ante_description/meshes/reader_bicep.stl" scale="1. 1. 1."/>
       </geometry>
+      <material name="green" />
     </visual>
   </link>
@@ -34,4 +36,5 @@
     <limit lower="-1.5707963" upper="1.5707963" effort="0." velocity="0."/>
   </joint>
+  <!-- create end effector link and joint -->
   <xacro:property name="elbow_offset_x" value="-0.02795" />
   <xacro:property name="elbow_offset_y" value="-0.00025" />
@@ -39,8 +42,10 @@
   <link name="reader_end_link">
     <visual>
+      <!-- the shoulder offset needs to be subtracted because the mesh is in the correct position before the offset -->
       <origin xyz="${-elbow_offset_x - shoulder_offset_x} ${-elbow_offset_y - shoulder_offset_y} ${-elbow_offset_z - shoulder_offset_z}" rpy="0 0 0" />
       <geometry>
         <mesh filename="package://ante_description/meshes/reader_end.stl" scale="1. 1. 1."/>
       </geometry>
+      <material name="green" />
     </visual>
   </link>

File: ante_description/parts/simple_wheel.xacro (robot description, xacro)
@@ -7,4 +7,5 @@
         <mesh filename="package://ante_description/meshes/simple_wheel.stl" scale="1. 1. 1."/>
       </geometry>
+      <material name="yellow" />
     </visual>
     <collision>

File: ante_description/robots/ante.urdf.xacro (robot description, xacro)
@@ -7,5 +7,7 @@
     <xacro:include filename="$(find ante_description)/parts/simple_wheel.xacro" />
     <xacro:include filename="$(find ante_description)/parts/reader_arm.xacro" />
+    <xacro:include filename="$(find ante_description)/parts/knob_wheel.xacro" />
     <!-- <xacro:include filename="$(find ante_description)/urdf/ros2_control.xacro" /> -->
+    <xacro:include filename="$(find ante_description)/util/materials.xacro" />
     <!-- create base_link -->
     <link name="base_link" />
@@ -52,5 +54,8 @@
     </xacro:solenoids>
     <xacro:reader_arm parent="chassis_link">
-        <origin xyz="0 0 0.2" rpy="0 0 0" />
+        <origin xyz="0 0 0.1" rpy="0 0 0" />
     </xacro:reader_arm>
+    <xacro:knob_wheel parent="chassis_link">
+        <origin xyz="0.138 0.072 0.115" rpy="0 -1.570796 0"/>
+    </xacro:knob_wheel>
 </robot>
