Commit message: forward position controller and readme

File: ante_description/parts/ros2_control.xacro (robot description, xacro)
@@ -1,5 +1,5 @@
 <?xml version="1.0" ?>
 <robot xmlns:xacro="http://www.ros.org/wiki/xacro">
-<xacro:macro name="ros2_control" params="prefix ros2_control_hardware_type usb_port">
+<xacro:macro name="ros2_control" params="ros2_control_hardware_type usb_port">
     <ros2_control name="ante" type="system">
         <hardware>
@@ -12,5 +12,21 @@
             </xacro:if>
         </hardware>
+        <joint name="reader_shoulder_joint">
+            <param name="initial_position">0.0</param>
+            <param name="id">1</param>
+            <param name="offset">0</param>
+            <command_interface name="position" />
+            <state_interface name="position" />
+            <state_interface name="velocity" />
+        </joint>
+        <joint name="reader_elbow_joint">
+            <param name="initial_position">0.0</param>
+            <param name="id">2</param>
+            <param name="offset">0</param>
+            <command_interface name="position" />
+            <state_interface name="position" />
+            <state_interface name="velocity" />
+        </joint>
     </ros2_control>
-</macro>
+</xacro:macro>
 </robot>

File: ante_description/robots/ante.urdf.xacro (robot description, xacro)
@@ -8,5 +8,5 @@
     <xacro:include filename="$(find ante_description)/parts/reader_arm.xacro" />
     <xacro:include filename="$(find ante_description)/parts/knob_wheel.xacro" />
-    <!-- <xacro:include filename="$(find ante_description)/urdf/ros2_control.xacro" /> -->
+    <xacro:include filename="$(find ante_description)/parts/ros2_control.xacro" />
     <xacro:include filename="$(find ante_description)/util/materials.xacro" />
     <!-- create base_link -->
@@ -59,3 +59,4 @@
         <origin xyz="0.138 0.072 0.115" rpy="0 -1.570796 0"/>
     </xacro:knob_wheel>
+    <xacro:ros2_control ros2_control_hardware_type="real" usb_port="/dev/ttyACM0"/>
 </robot>
