Commit message: updated reader arm urdf

File: ante_description/parts/reader_arm.xacro (robot description, xacro)
@@ -17,12 +17,9 @@
   </joint>
   <!-- create bicep and shoulder joint -->
-  <xacro:property name="shoulder_offset_x" value="-0.005611" />
-  <xacro:property name="shoulder_offset_y" value="0.012795" />
-  <xacro:property name="shoulder_offset_z" value="0.0442" />
-  <link name="reader_bicep_link">
+  <link name="reader_upper_link">
     <visual>
-      <origin xyz="${-shoulder_offset_x} ${-shoulder_offset_y} ${-shoulder_offset_z}" rpy="0 0 0" />
+      <origin xyz="0 0 0" rpy="0 0 0" />
       <geometry>
-        <mesh filename="package://ante_description/meshes/reader_bicep.stl" scale="1. 1. 1."/>
+        <mesh filename="package://ante_description/meshes/reader_upper.stl" scale="1. 1. 1."/>
       </geometry>
       <material name="green" />
@@ -30,20 +27,19 @@
   </link>
   <joint name="reader_shoulder_joint" type="revolute">
-    <origin xyz="${shoulder_offset_x} ${shoulder_offset_y} ${shoulder_offset_z}" rpy="0 0 0"/>
+    <origin xyz="0 0 0" rpy="0 0 0"/>
     <parent link="reader_base_link"/>
-    <child link="reader_bicep_link"/>
+    <child link="reader_upper_link"/>
     <axis xyz="0 1 0."/>
-    <limit lower="-1.5707963" upper="1.5707963" effort="0." velocity="0."/>
+    <limit lower="0" upper="3.1416" effort="0." velocity="0."/>
   </joint>
   <!-- create end effector link and joint -->
-  <xacro:property name="elbow_offset_x" value="-0.02795" />
-  <xacro:property name="elbow_offset_y" value="-0.00025" />
-  <xacro:property name="elbow_offset_z" value="0.160527" />
-  <link name="reader_end_link">
+  <xacro:property name="lower_offset_x" value="-0.160943" />
+  <xacro:property name="lower_offset_y" value="0.0" />
+  <xacro:property name="lower_offset_z" value="0.02795" />
+  <link name="reader_lower_link">
     <visual>
-      <!-- the shoulder offset needs to be subtracted because the mesh is in the correct position before the offset -->
-      <origin xyz="${-elbow_offset_x - shoulder_offset_x} ${-elbow_offset_y - shoulder_offset_y} ${-elbow_offset_z - shoulder_offset_z}" rpy="0 0 0" />
+      <origin xyz="0 0 0" rpy="0 0 0" />
       <geometry>
-        <mesh filename="package://ante_description/meshes/reader_end.stl" scale="1. 1. 1."/>
+        <mesh filename="package://ante_description/meshes/reader_lower.stl" scale="1. 1. 1."/>
       </geometry>
       <material name="green" />
@@ -51,9 +47,9 @@
   </link>
   <joint name="reader_elbow_joint" type="revolute">
-    <origin xyz="${elbow_offset_x} ${elbow_offset_y} ${elbow_offset_z}" rpy="0 0 0"/>
-    <parent link="reader_bicep_link"/>
-    <child link="reader_end_link"/>
+    <origin xyz="${lower_offset_x} ${lower_offset_y} ${lower_offset_z}" rpy="0 0 0"/>
+    <parent link="reader_upper_link"/>
+    <child link="reader_lower_link"/>
     <axis xyz="0 1 0."/>
-    <limit lower="-1.5707963" upper="1.5707963" effort="0." velocity="0."/>
+    <limit lower="0" upper="3.1416" effort="0." velocity="0."/>
   </joint>
 </xacro:macro>

File: ante_description/robots/ante.urdf.xacro (robot description, xacro)
@@ -13,5 +13,5 @@
     <link name="base_link" />
     <xacro:drivebase parent="base_link">
-        <origin xyz="0 0 0" rpy="0 0 0"/>
+        <origin xyz="0 0 0" rpy="0 0 1.570796"/>
     </xacro:drivebase>
     <xacro:simple_wheel
@@ -54,5 +54,5 @@
     </xacro:solenoids>
     <xacro:reader_arm parent="chassis_link">
-        <origin xyz="0 0 0.1" rpy="0 0 0" />
+        <origin xyz="0 0 0.2" rpy="0 0 0" />
     </xacro:reader_arm>
     <xacro:knob_wheel parent="chassis_link">
